Commit message: unifytips0.5: modify the IK for robocasa mujoco benchmark

File: gr00t/eval/robot_assets/GR1T2/urdf/GR1T2_fourier_hand_6dof.urdf (robot description, URDF)
Before this commit: robot GR1T2_fourier_hand_6dof, 71 links, 70 joints
Joints:
- joint left_elbow_pitch_joint: limit lower=-2.27 upper=2.27 effort=30 velocity=7.33 -> lower=-3.0 upper=0.0 effort=30 velocity=7.33
- joint left_shoulder_pitch_joint: limit lower=-2.79 upper=1.92 effort=38 velocity=9.11 -> lower=-3.0 upper=3.0 effort=38 velocity=9.11
- joint left_shoulder_roll_joint: limit lower=-0.57 upper=2.53 effort=38 velocity=9.11 -> lower=0.0 upper=3.0 effort=38 velocity=9.11
- joint left_shoulder_yaw_joint: limit lower=-2.97 upper=2.97 effort=30 velocity=7.33 -> lower=-3.0 upper=3.0 effort=30 velocity=7.33
- joint left_wrist_pitch_joint: limit lower=-0.61 upper=0.61 effort=3.95 velocity=27.96 -> lower=-1.5 upper=1.5 effort=3.95 velocity=27.96
- joint left_wrist_roll_joint: limit lower=-0.87 upper=0.96 effort=3.95 velocity=27.96 -> lower=-3.0 upper=3.0 effort=3.95 velocity=27.96
- joint left_wrist_yaw_joint: limit lower=-2.97 upper=2.97 effort=10.2 velocity=24.4 -> lower=-3.0 upper=3.0 effort=10.2 velocity=24.4
- joint right_elbow_pitch_joint: limit lower=-2.27 upper=2.27 effort=30 velocity=7.33 -> lower=-3.0 upper=0.0 effort=30 velocity=7.33
- joint right_shoulder_pitch_joint: limit lower=-2.79 upper=1.92 effort=38 velocity=9.11 -> lower=-3.0 upper=3.0 effort=38 velocity=9.11
- joint right_shoulder_roll_joint: limit lower=-2.53 upper=0.57 effort=38 velocity=9.11 -> lower=-3.0 upper=0.0 effort=38 velocity=9.11
- joint right_shoulder_yaw_joint: limit lower=-2.97 upper=2.97 effort=30 velocity=7.33 -> lower=-3.0 upper=3.0 effort=30 velocity=7.33
- joint right_wrist_pitch_joint: limit lower=-0.61 upper=0.61 effort=3.95 velocity=27.96 -> lower=-3.0 upper=3.0 effort=3.95 velocity=27.96
- joint right_wrist_roll_joint: limit lower=-0.96 upper=0.87 effort=3.95 velocity=27.96 -> lower=-3.0 upper=3.0 effort=3.95 velocity=27.96
- joint right_wrist_yaw_joint: limit lower=-2.97 upper=2.97 effort=10.2 velocity=24.4 -> lower=-3.0 upper=3.0 effort=10.2 velocity=24.4

Commit message: unifytips0.5: modify the tip keypoints dataset V4 and finger commands for retarget

File: gr00t/eval/robot_assets/GR1T2/urdf/GR1T2_fourier_hand_6dof.urdf (robot description, URDF)
Before this commit: robot GR1T2_fourier_hand_6dof, 71 links, 70 joints
Joints:
- joint right_wrist_pitch_joint: limit lower=-3.0 upper=3.0 effort=3.95 velocity=27.96 -> lower=-1.5 upper=1.5 effort=3.95 velocity=27.96
