Commit message: unifytips0.5:modify the tip keypoints dataset V5 and retarget api

File: gr00t/eval/robot_assets/fourier_hand/fourier_left_hand_glb copy.urdf (robot description, URDF)
Before this commit: robot fourier_left_hand_6dof, 17 links, 16 joints
Joints:
- joint L_index_intermediate_joint: mimic joint=L_index_proximal_joint multiplier=1 offset=0 -> joint=L_index_proximal_joint multiplier=1.128 offset=0
- joint L_middle_intermediate_joint: mimic joint=L_middle_proximal_joint multiplier=1 offset=0 -> joint=L_middle_proximal_joint multiplier=1.131 offset=0
- joint L_pinky_intermediate_joint: mimic joint=L_pinky_proximal_joint multiplier=1 offset=0 -> joint=L_pinky_proximal_joint multiplier=1.129 offset=0
- joint L_ring_intermediate_joint: mimic joint=L_ring_proximal_joint multiplier=1 offset=0 -> joint=L_ring_proximal_joint multiplier=1.143 offset=0
- joint L_thumb_distal_joint: mimic joint=L_thumb_proximal_pitch_joint multiplier=1 offset=0 -> joint=L_thumb_proximal_pitch_joint multiplier=0.974 offset=0

File: gr00t/eval/robot_assets/fourier_hand/fourier_left_hand_glb.urdf (robot description, URDF)
Before this commit: robot fourier_left_hand_6dof, 17 links, 16 joints
Joints:
- joint L_index_intermediate_joint: mimic joint=L_index_proximal_joint multiplier=1.128 offset=0 -> joint=L_index_proximal_joint multiplier=1 offset=0
- joint L_middle_intermediate_joint: mimic joint=L_middle_proximal_joint multiplier=1.131 offset=0 -> joint=L_middle_proximal_joint multiplier=1 offset=0
- joint L_pinky_intermediate_joint: mimic joint=L_pinky_proximal_joint multiplier=1.129 offset=0 -> joint=L_pinky_proximal_joint multiplier=1 offset=0
- joint L_ring_intermediate_joint: mimic joint=L_ring_proximal_joint multiplier=1.143 offset=0 -> joint=L_ring_proximal_joint multiplier=1 offset=0
- joint L_thumb_distal_joint: mimic joint=L_thumb_proximal_pitch_joint multiplier=0.974 offset=0 -> joint=L_thumb_proximal_pitch_joint multiplier=1 offset=0

File: gr00t/eval/robot_assets/fourier_hand/fourier_right_hand_glb copy.urdf (robot description, URDF)
Before this commit: robot fourier_left_hand_6dof, 17 links, 16 joints
Links:
- removed link L_hand_base_link
- removed link L_index_intermediate_link
- removed link L_index_proximal_link
- removed link L_index_tip_link
- removed link L_middle_intermediate_link
- removed link L_middle_proximal_link
- removed link L_middle_tip_link
- removed link L_pinky_intermediate_link
- removed link L_pinky_proximal_link
- removed link L_pinky_tip_link
- removed link L_ring_intermediate_link
- removed link L_ring_proximal_link
- removed link L_ring_tip_link
- removed link L_thumb_distal_link
- removed link L_thumb_proximal_base_link
- removed link L_thumb_proximal_link
- removed link L_thumb_tip_link
- added link R_hand_base_link, mass 0.306; collision mesh filename=meshes/fourier_hand_6dof/R_hand_base_link.STL; visual mesh filename=meshes/fourier_hand_6dof/R_hand_base_link.STL
- added link R_index_intermediate_link, mass 0.01292544; collision mesh filename=meshes/fourier_hand_6dof/R_index_intermediate_link.STL; visual mesh filename=meshes/fourier_hand_6dof/R_index_intermediate_link.STL
- added link R_index_proximal_link, mass 0.01911771; collision mesh filename=meshes/fourier_hand_6dof/R_index_proximal_link.STL; visual mesh filename=meshes/fourier_hand_6dof/R_index_proximal_link.STL
- added link R_index_tip_link; visual sphere radius=0.005
- added link R_middle_intermediate_link, mass 0.01535; collision mesh filename=meshes/fourier_hand_6dof/R_middle_intermediate_link.STL; visual mesh filename=meshes/fourier_hand_6dof/R_middle_intermediate_link.STL
- added link R_middle_proximal_link, mass 0.01911771; collision mesh filename=meshes/fourier_hand_6dof/R_middle_proximal_link.STL; visual mesh filename=meshes/fourier_hand_6dof/R_middle_proximal_link.STL
- added link R_middle_tip_link; visual sphere radius=0.005
- added link R_pinky_intermediate_link, mass 0.00568707; collision mesh filename=meshes/fourier_hand_6dof/R_pinky_intermediate_link.STL; visual mesh filename=meshes/fourier_hand_6dof/R_pinky_intermediate_link.STL
- added link R_pinky_proximal_link, mass 0.01911771; collision mesh filename=meshes/fourier_hand_6dof/R_pinky_proximal_link.STL; visual mesh filename=meshes/fourier_hand_6dof/R_pinky_proximal_link.STL
- added link R_pinky_tip_link; visual sphere radius=0.005
- added link R_ring_intermediate_link, mass 0.012925; collision mesh filename=meshes/fourier_hand_6dof/R_ring_intermediate_link.STL; visual mesh filename=meshes/fourier_hand_6dof/R_ring_intermediate_link.STL
- added link R_ring_proximal_link, mass 0.01911771; collision mesh filename=meshes/fourier_hand_6dof/R_ring_proximal_link.STL; visual mesh filename=meshes/fourier_hand_6dof/R_ring_proximal_link.STL
- added link R_ring_tip_link; visual sphere radius=0.005
- added link R_thumb_distal_link, mass 0.01974135; collision mesh filename=meshes/fourier_hand_6dof/R_thumb_distal_link.STL; visual mesh filename=meshes/fourier_hand_6dof/R_thumb_distal_link.STL
- added link R_thumb_proximal_base_link, mass 0.00948218; collision mesh filename=meshes/fourier_hand_6dof/R_thumb_proximal_base_link.STL; visual mesh filename=meshes/fourier_hand_6dof/R_thumb_proximal_base_link.STL
- added link R_thumb_proximal_link, mass 0.07405243; collision mesh filename=meshes/fourier_hand_6dof/R_thumb_proximal_link.STL; visual mesh filename=meshes/fourier_hand_6dof/R_thumb_proximal_link.STL
- added link R_thumb_tip_link; visual sphere radius=0.005
Joints:
- removed joint L_index_intermediate_joint
- removed joint L_index_proximal_joint
- removed joint L_index_tip_joint
- removed joint L_middle_intermediate_joint
- removed joint L_middle_proximal_joint
- removed joint L_middle_tip_joint
- removed joint L_pinky_intermediate_joint
- removed joint L_pinky_proximal_joint
- removed joint L_pinky_tip_joint
- removed joint L_ring_intermediate_joint
- removed joint L_ring_proximal_joint
- removed joint L_ring_tip_joint
- removed joint L_thumb_distal_joint
- removed joint L_thumb_proximal_pitch_joint
- removed joint L_thumb_proximal_yaw_joint
- removed joint L_thumb_tip_joint
- added joint R_index_intermediate_joint: type revolute, parent R_index_proximal_link, child R_index_intermediate_link, origin xyz=0.031532 -0.0054551 0 rpy=0 0 0, axis 0 0 1, limit lower=-1.74 upper=0 effort=10 velocity=0.8, mimic joint=R_index_proximal_joint multiplier=1.128 offset=0
- added joint R_index_proximal_joint: type revolute, parent R_hand_base_link, child R_index_proximal_link, origin xyz=0.026864 0.012307 -0.095892 rpy=-3.1403 1.5184 0.0013039, axis 0 0 1, limit lower=-1.57 upper=0 effort=10 velocity=0.8
- added joint R_index_tip_joint: type fixed, parent R_index_intermediate_link, child R_index_tip_link, origin xyz=0.038 -0.0015 0 rpy=0 0 0
- added joint R_middle_intermediate_joint: type revolute, parent R_middle_proximal_link, child R_middle_intermediate_link, origin xyz=0.031662 -0.0046408 0 rpy=0 0 0, axis 0 0 1, limit lower=-1.74 upper=0 effort=10 velocity=0.8, mimic joint=R_middle_proximal_joint multiplier=1.131 offset=0
- added joint R_middle_proximal_joint: type revolute, parent R_hand_base_link, child R_middle_proximal_link, origin xyz=0.0084962 0.012307 -0.097896 rpy=-1.7476 1.5707 1.394, axis 0 0 1, limit lower=-1.57 upper=0 effort=10 velocity=0.8
- added joint R_middle_tip_joint: type fixed, parent R_middle_intermediate_link, child R_middle_tip_link, origin xyz=0.045 0.0005 0 rpy=0 0 0
- added joint R_pinky_intermediate_joint: type revolute, parent R_pinky_proximal_link, child R_pinky_intermediate_link, origin xyz=0.031338 -0.0064763 0 rpy=0 0 6.7976E-05, axis 0 0 1, limit lower=-1.74 upper=0 effort=10 velocity=0.8, mimic joint=R_pinky_proximal_joint multiplier=1.129 offset=0
- added joint R_pinky_proximal_joint: type revolute, parent R_hand_base_link, child R_pinky_proximal_link, origin xyz=-0.028232 0.012307 -0.095916 rpy=-0.00065397 1.4661 3.1409, axis 0 0 1, limit lower=-1.57 upper=0 effort=10 velocity=0.8
- added joint R_pinky_tip_joint: type fixed, parent R_pinky_intermediate_link, child R_pinky_tip_link, origin xyz=0.031 -0.004 0 rpy=0 0 0
- added joint R_ring_intermediate_joint: type revolute, parent R_ring_proximal_link, child R_ring_intermediate_link, origin xyz=0.031531 -0.0054572 0 rpy=0 0 0, axis 0 0 1, limit lower=-1.74 upper=0 effort=10 velocity=0.8, mimic joint=R_ring_proximal_joint multiplier=1.143 offset=0
- added joint R_ring_proximal_joint: type revolute, parent R_hand_base_link, child R_ring_proximal_link, origin xyz=-0.009965 0.012307 -0.097841 rpy=0 1.5184 3.1416, axis 0 0 1, limit lower=-1.57 upper=0 effort=10 velocity=0.8
- added joint R_ring_tip_joint: type fixed, parent R_ring_intermediate_link, child R_ring_tip_link, origin xyz=0.038 -0.0015 0 rpy=0 0 0
- added joint R_thumb_distal_joint: type revolute, parent R_thumb_proximal_link, child R_thumb_distal_link, origin xyz=0.061444 0.0082822 0 rpy=0 0 1.221E-05, axis 0 0 1, limit lower=0 upper=1.23 effort=10 velocity=0.8, mimic joint=R_thumb_proximal_pitch_joint multiplier=0.974 offset=0
- added joint R_thumb_proximal_pitch_joint: type revolute, parent R_thumb_proximal_base_link, child R_thumb_proximal_link, origin xyz=0.02175 0 0 rpy=1.5709 1.221E-05 0, axis 0 0 1, limit lower=0 upper=1.22 effort=10 velocity=0.8
- added joint R_thumb_proximal_yaw_joint: type revolute, parent R_hand_base_link, child R_thumb_proximal_base_link, origin xyz=0.021995 0.015502 -0.024995 rpy=3.1416 0 0, axis 0 0 1, limit lower=-1.74 upper=0 effort=10 velocity=0.8
- added joint R_thumb_tip_joint: type fixed, parent R_thumb_distal_link, child R_thumb_tip_link, origin xyz=0.031 0 0 rpy=0 0 0
